File: board/CurrentSensorV1/CurrentSensorV1.sch (KiCad schematic (older format))
At the start: 17 parts, among them J1 USB_B_Micro, J2 FTDI_Header, J3 AudioJack3_GroundPinNumbers, J4 0, J5 0, J6 Conn_01x02_Female, J7 Conn_01x02_Female, SW2 SW_SPST_SM_DP, SW3 SW_SPST_SM_DP, U1 UA78M05CDCY, U2 ESP-01v090, U3 ADS1115

Commit message: Starting v4
Parts:
- removed C1: 0.1uF, Capacitor_THT:C_Disc_D3.0mm_W1.6mm_P2.50mm, symbol Device:CP
- removed C3: 0.33uF, Capacitor_THT:C_Disc_D3.0mm_W1.6mm_P2.50mm, symbol Device:CP
- removed J4, J5: 0, Connector_PinHeader_2.54mm:PinHeader_1x04_P2.54mm_Vertical, symbol Connector:Conn_01x04_Female
- removed R4: R, Resistor_THT:R_Axial_DIN0204_L3.6mm_D1.6mm_P7.62mm_Horizontal, symbol Device:R
- removed U1: UA78M05CDCY, UA78M05CDCY:SOT230P700X180-4N, symbol UA78M05CDCY:UA78M05CDCY
- removed U3: ADS1115, Connector_PinHeader_2.54mm:PinHeader_1x10_P2.54mm_Vertical, symbol ADS1115:ADS1115
- added C1, C3, C5: 1uF, Capacitor_SMD:C_0402_1005Metric, symbol Device:C
- added C4: 1000uF, Capacitor_SMD:C_Elec_8x10.2, symbol Device:CP
- added C6: 2.2uF, Capacitor_SMD:C_0603_1608Metric, symbol Device:C
- added D1: D, Diode_SMD:D_SOD-123, symbol Device:D
- added FB1, FB2: Ferrite_Bead, Resistor_SMD:R_0805_2012Metric, symbol Device:Ferrite_Bead
- added H1, H2, H3, H4: MountingHole_Pad, MountingHole:MountingHole_2.5mm_Pad, symbol Mechanical:MountingHole_Pad
- added J8: AudioJack3_GroundPinNumbers, audio35mm:Tayda_3.5mm_stereo_TRS_jack_A-853, symbol JACK_TRS:AudioJack3_GroundPinNumbers
- added R1, R2, R3, R6: 10K, Resistor_SMD:R_0603_1608Metric, symbol Device:R
- added R5: 680R, Resistor_SMD:R_0603_1608Metric, symbol Device:R
- added TP2, TP3: TestPoint, Connector_PinSocket_2.54mm:PinSocket_1x01_P2.54mm_Vertical, symbol Connector:TestPoint
- added U1: ADS1015_IC, Package_SO:VSSOP-10_3x3mm_P0.5mm, symbol ADS1115:ADS1015_IC
- added U3: AMS1117-3.3, Package_TO_SOT_SMD:SOT-223-3_TabPin2, symbol Regulator_Linear:AMS1117-3.3
- C2: value 470uF -> 100uF; footprint Capacitor_THT:CP_Radial_D5.0mm_P2.00mm -> Capacitor_Tantalum_SMD:CP_EIA-3528-12_Kemet-T; JLCPCB_CORRECTION (none) -> 0;0;180; LCSC (none) -> C16133
- FLASH1: renamed from SW3; LCSC (none) -> C530667
- RST1: renamed from SW2; LCSC (none) -> C530667
Connections:
- net +3V3: now also C3.1, C4.1, C5.2, D1.1 (K), R1.1, R2.1, R6.1, TP2.1, U1.8 (VDD), U3.2 (VO)
- net GND: now also J1.6 (Shield), C3.2, C4.2, C5.1, FB1.2, H1.1, H2.1, H3.1, H4.1, R3.1, R5.1, TP3.1, U1.1 (ADDR), U1.3 (GND), U3.1 (GND)
- net SCL: now also R1.2, U1.10 (SCL)
- net SDA: now also R2.2, U1.9 (SDA)
- net VBUS: now also FB2.2, U3.3 (VI)
- net FTDI_RX: now reaches J2.2 (RX), U2.1 (UTXD)
- net RST: now reaches RST1.1 (A), RST1.2 (A), U2.5 (RST)
- net RST: now also C6.1, D1.2 (A), R6.2
- net FTDI_TX: now reaches J2.3 (TX), U2.8 (URXD)
- net at J2.1 (DTR): now also C6.2, R5.2
- net AIN3: now reaches J7.1 (Pin_1)
- net AIN3: now also J8.3 (T), U1.7 (AIN3)
- net AIN2: now reaches J7.2 (Pin_2)
- net AIN2: now also J8.1 (S), U1.6 (AIN2)
- net AIN0: now reaches J3.1 (S), J6.2 (Pin_2)
- net AIN0: now also U1.4 (AIN0)
- net AIN1: now reaches J3.3 (T), J6.1 (Pin_1)
- net AIN1: now also U1.5 (AIN1)
- new net: C1.1, FB2.1
- new net: C1.2, FB1.1
- new net ALERT: R3.2, U1.2 (ALERT)
Other:
- moved on the sheet: C2, FLASH1, J2, J3, J6, J7, RST1, TP1, U2

Commit message: Working on V4
Parts:
- removed C2: 100uF, Capacitor_Tantalum_SMD:CP_EIA-3528-12_Kemet-T, symbol Device:C
- removed C6: 2.2uF, Capacitor_SMD:C_0603_1608Metric, symbol Device:C
- removed D1: D, Diode_SMD:D_SOD-123, symbol Device:D
- removed FB1, FB2: Ferrite_Bead, Resistor_SMD:R_0805_2012Metric, symbol Device:Ferrite_Bead
- removed FLASH1, RST1: SW_SPST_SM_DP, eec:E-Switch-TL3342F160QG-0, symbol ADS1115:SW_SPST_SM_DP
- removed J1: USB_B_Micro, digikey-footprints:USB_Micro_AB_Female_0475890001_DP_PWR_GND, symbol Connector:USB_B_Micro
- removed J2: FTDI_Header, avr-arduino:FTDI_Header, symbol avr-arduino:FTDI_Header
- removed R5: 680R, Resistor_SMD:R_0603_1608Metric, symbol Device:R
- removed TP3: TestPoint, Connector_PinSocket_2.54mm:PinSocket_1x01_P2.54mm_Vertical, symbol Connector:TestPoint
- added J2: ESP_Header_DP, avr-arduino:FTDI_Header, symbol avr-arduino:ESP_Header_DP
- added U9: USB_B_Micro, CurrentSensorV1:USB_MICRO_M5SS_DP, symbol usb_b_micro_8_pads:USB_B_Micro
Connections:
- net +3V3: now also J2.4 (VCC)
- net FTDI_RX: now also J2.2 (RX)
- net FTDI_TX: now also J2.3 (TX)
- net GND: now also C1.2, J2.6 (GND), U9.5 (GND), U9.6 (Shield), U9.7 (Shield), U9.8 (Shield), U9.9 (Shield)
- net RST: now also J2.1 (RTS)
- net SDA: now also J2.5 (GPIO0)
- net VBUS: now also C1.1, U9.1 (VBUS)
Other:
- moved on the sheet: C4, C5, H1, H2, H3, H4, J3, J6, R1, R2, R3, R6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

Commit message: V4
Parts:
- C1, C3, C5: symbol Device:C -> CurrentSensorV1-rescue:C-Device
- C4: symbol Device:CP -> CurrentSensorV1-rescue:CP-Device
- H1, H2, H3, H4: symbol Mechanical:MountingHole_Pad -> CurrentSensorV1-rescue:MountingHole_Pad-Mechanical
- J2: symbol avr-arduino:ESP_Header_DP -> CurrentSensorV1-rescue:ESP_Header_DP-avr-arduino
- J6, J7: symbol Connector:Conn_01x02_Female -> CurrentSensorV1-rescue:Conn_01x02_Female-Connector
- R1, R2, R3, R6: symbol Device:R -> CurrentSensorV1-rescue:R-Device
- TP1, TP2: symbol Connector:TestPoint -> CurrentSensorV1-rescue:TestPoint-Connector
- U2: symbol ESP8266:ESP-01v090 -> CurrentSensorV1-rescue:ESP-01v090-ESP8266
- U3: symbol Regulator_Linear:AMS1117-3.3 -> CurrentSensorV1-rescue:AMS1117-3.3-Regulator_Linear
- U9: symbol usb_b_micro_8_pads:USB_B_Micro -> CurrentSensorV1-rescue:USB_B_Micro-usb_b_micro_8_pads
Changed lines of the file:
@@
 $EndDescr
 $Comp
-L power:GND #PWR0101
+L CurrentSensorV1-rescue:GND-power #PWR0101
 U 1 1 5F67F747
 P 850 4300
@@
 $EndComp
 $Comp
-L power:+3.3V #PWR0102
+L CurrentSensorV1-rescue:+3.3V-power #PWR0102
 U 1 1 5F6850CC
 P 5600 2700
@@
 $EndComp
 $Comp
-L power:+3.3V #PWR0103
+L CurrentSensorV1-rescue:+3.3V-power #PWR0103
 U 1 1 5F68586F
 P 4600 2750
@@
 $EndComp
 $Comp
-L power:GND #PWR0104
+L CurrentSensorV1-rescue:GND-power #PWR0104
 U 1 1 5F686DB3
 P 5400 2700
@@
 $EndComp
 $Comp
-L power:GND #PWR0107
+L CurrentSensorV1-rescue:GND-power #PWR0107
 U 1 1 5F69179D
 P 1250 2450
@@
 $EndComp
 $Comp
-L power:+3.3V #PWR0108
+L CurrentSensorV1-rescue:+3.3V-power #PWR0108
 U 1 1 5F691A9F
 P 1550 2450
@@
 $EndComp
 $Comp
-L power:VBUS #PWR0110
+L CurrentSensorV1-rescue:VBUS-power #PWR0110
 U 1 1 5F6B3D4C
 P 1400 3550
@@
 	6900 1000 6900 1200
 $Comp
-L Connector:Conn_01x02_Female J6
+L CurrentSensorV1-rescue:Conn_01x02_Female-Connector J6
 U 1 1 5F6955DB
 P 5200 1700
@@
 	5400 1000 5450 1000
 $Comp
-L power:GND #PWR0109
+L CurrentSensorV1-rescue:GND-power #PWR0109
 U 1 1 5F757012
 P 1250 1100
@@
 $EndComp
 $Comp
-L power:VBUS #PWR0113
+L CurrentSensorV1-rescue:VBUS-power #PWR0113
 U 1 1 5F7576FC
 P 1550 1100
@@
 $EndComp
 $Comp
-L power:GND #PWR0114
+L CurrentSensorV1-rescue:GND-power #PWR0114
 U 1 1 5F75ED44
 P 2500 3150
@@
 	2500 3100 2500 3150
 $Comp
-L power:+3.3V #PWR0111
+L CurrentSensorV1-rescue:+3.3V-power #PWR0111
 U 1 1 5F785201
 P 2700 1000
@@
 $EndComp
 $Comp
-L power:VBUS #PWR0117
+L CurrentSensorV1-rescue:VBUS-power #PWR0117
 U 1 1 5F787AC4
 P 3200 950
@@
 $EndComp
 $Comp
-L power:GND #PWR0118
+L CurrentSensorV1-rescue:GND-power #PWR0118
 U 1 1 5F79B4F5
 P 2800 2150
@@
 	5400 2700 5400 2600
 $Comp
-L power:VBUS #PWR0119
+L CurrentSensorV1-rescue:VBUS-power #PWR0119
 U 1 1 5F7CF7D9
 P 2350 1700
@@
 $EndComp
 $Comp
-L power:+3.3V #PWR0120
+L CurrentSensorV1-rescue:+3.3V-power #PWR0120
 U 1 1 5F7CFF2C
 P 3250 1700
@@
 	5700 3000 5700 2600
 $Comp
-L Connector:TestPoint TP1
+L CurrentSensorV1-rescue:TestPoint-Connector TP1
 U 1 1 5F834784
 P 3200 800
@@
 $EndComp
 $Comp
-L power:+3.3V #PWR0115
+L CurrentSensorV1-rescue:+3.3V-power #PWR0115
 U 1 1 6037FDE9
 P 6150 2350
@@
 $EndComp
 $Comp
-L Device:R R6
+L CurrentSensorV1-rescue:R-Device R6
 U 1 1 6038053A
 P 6150 2600
@@
 $EndComp
 $Comp
-L Device:C C5
+L CurrentSensorV1-rescue:C-Device C5
 U 1 1 6037AC9B
 P 2750 4000
@@
 $EndComp
 $Comp
-L power:+3.3V #PWR0116
+L CurrentSensorV1-rescue:+3.3V-power #PWR0116
 U 1 1 6037D07E
 P 3000 4150
@@
 $EndComp
 $Comp
-L power:GND #PWR0121
+L CurrentSensorV1-rescue:GND-power #PWR0121
 U 1 1 6038225E
 P 2750 3650
@@
 $EndComp
 $Comp
-L Device:R R2
+L CurrentSensorV1-rescue:R-Device R2
 U 1 1 603858DC
 P 3050 4450
@@
 $EndComp
 $Comp
-L Device:R R1
+L CurrentSensorV1-rescue:R-Device R1
 U 1 1 60385015
 P 3050 4350
@@
 $EndComp
 $Comp
-L power:+3.3V #PWR0122
+L CurrentSensorV1-rescue:+3.3V-power #PWR0122
 U 1 1 6039C899
 P 3350 4350
@@
 $EndComp
 $Comp
-L power:+3.3V #PWR0123
+L CurrentSensorV1-rescue:+3.3V-power #PWR0123
 U 1 1 6039D0F2
 P 3350 4450
@@
 	3200 4450 3350 4450
 $Comp
-L power:GND #PWR0124
+L CurrentSensorV1-rescue:GND-power #PWR0124
 U 1 1 603A27AC
 P 2800 4750
@@
 ALERT
 $Comp
-L Device:R R3
+L CurrentSensorV1-rescue:R-Device R3
 U 1 1 603CACB2
 P 3050 4650
@@
 	2600 4650 2900 4650
 $Comp
-L Connector:Conn_01x02_Female J7
+L CurrentSensorV1-rescue:Conn_01x02_Female-Connector J7
 U 1 1 5F694DC9
 P 6900 1400
@@
 Connection ~ 6900 1000
 $Comp
-L power:GND #PWR0125
+L CurrentSensorV1-rescue:GND-power #PWR0125
 U 1 1 604346D4
 P 3000 4550
@@
 	3200 800  3200 950
 $Comp
-L Connector:TestPoint TP2
+L CurrentSensorV1-rescue:TestPoint-Connector TP2
 U 1 1 6047E08F
 P 2700 800
@@
 	2700 800  2700 1000
 $Comp
-L power:GND #PWR0126
+L CurrentSensorV1-rescue:GND-power #PWR0126
 U 1 1 604AA4F9
 P 3350 4650
@@
 RST
 $Comp
-L power:+3.3V #PWR0128
+L CurrentSensorV1-rescue:+3.3V-power #PWR0128
 U 1 1 6057E04E
 P 4800 3000
@@
 	4500 2750 4600 2750
 $Comp
-L Device:CP C4
+L CurrentSensorV1-rescue:CP-Device C4
 U 1 1 6060DF74
 P 1400 2200
@@
 $EndComp
 $Comp
-L Regulator_Linear:AMS1117-3.3 U3
+L CurrentSensorV1-rescue:AMS1117-3.3-Regulator_Linear U3
 U 1 1 60649B4D
 P 2800 1700
@@
 $EndComp
 $Comp
-L Device:C C3
+L CurrentSensorV1-rescue:C-Device C3
 U 1 1 60673198
 P 1400 1900
@@
 $EndComp
 $Comp
-L Device:C C1
+L CurrentSensorV1-rescue:C-Device C1
 U 1 1 606769FE
 P 1400 850
@@
 	4550 3100 4500 3100
 $Comp
-L ESP8266:ESP-01v090 U2
+L CurrentSensorV1-rescue:ESP-01v090-ESP8266 U2
 U 1 1 5F67B525
 P 3550 2950
@@
 $EndComp
 $Comp
-L Mechanical:MountingHole_Pad H1
+L CurrentSensorV1-rescue:MountingHole_Pad-Mechanical H1
 U 1 1 607BDB4C
 P 5000 3500
@@
 $EndComp
 $Comp
-L power:GND #PWR0127
+L CurrentSensorV1-rescue:GND-power #PWR0127
 U 1 1 607BF8E0
 P 5000 3750
@@
 	5000 3600 5000 3750
 $Comp
-L Mechanical:MountingHole_Pad H2
+L CurrentSensorV1-rescue:MountingHole_Pad-Mechanical H2
 U 1 1 607C4343
 P 5200 3750
@@
 $EndComp
 $Comp
-L power:GND #PWR0129
+L CurrentSensorV1-rescue:GND-power #PWR0129
 U 1 1 607C4349
 P 5200 4000
@@
 	5200 3850 5200 4000
 $Comp
-L Mechanical:MountingHole_Pad H3
+L CurrentSensorV1-rescue:MountingHole_Pad-Mechanical H3
 U 1 1 607C71AC
 P 5400 4000
@@
 $EndComp
 $Comp
-L power:GND #PWR0130
+L CurrentSensorV1-rescue:GND-power #PWR0130
 U 1 1 607C71B2
 P 5400 4250
@@
 	5400 4100 5400 4250
 $Comp
-L Mechanical:MountingHole_Pad H4
+L CurrentSensorV1-rescue:MountingHole_Pad-Mechanical H4
 U 1 1 607CA084
 P 5550 4250
@@
 $EndComp
 $Comp
-L power:GND #PWR0131
+L CurrentSensorV1-rescue:GND-power #PWR0131
 U 1 1 607CA08A
 P 5550 4500
@@
 	1550 850  1550 1100
 $Comp
-L avr-arduino:ESP_Header_DP J2
+L CurrentSensorV1-rescue:ESP_Header_DP-avr-arduino J2
 U 1 1 60A3E8A5
 P 5700 2400
@@
 	2750 3650 2750 3850
 $Comp
-L usb_b_micro_8_pads:USB_B_Micro U9
+L CurrentSensorV1-rescue:USB_B_Micro-usb_b_micro_8_pads U9
 U 1 1 609BBE83
 P 900 3750
